File: KEY/KEY.kicad_pcb (KiCad board)
At the start: 2 copper layers, 50 x 80 mm, 29 parts, among them J1 BUS, J3 FLASH/CONF, Q1 BC846, Q2 BC846, Q3 BC857, U1 AP63203WU, U2 WT8266-S1, U3 74LVC138

Commit message: Enhance PCB design
Parts:
- moved C2 2.74 mm to (126.7, 70.5)
- moved R5 0.52 mm to (138.5, 120.7)
- moved GND 0.14 mm to (133.9, 64.5)
- turned R2 to 180 degrees
- turned R4 to 90 degrees
Routing:
- net GND: track 229.4 -> 99.6 mm, vias 4 -> 2
- net +3.3V: track 158.7 -> 150.3 mm, vias 9 -> 3
- net TX: track 100.2 -> 106.2 mm
- net +12V: track 145.2 -> 140.8 mm
- net Net-(J5-Pin_4): track 14.9 -> 11.5 mm
- net Net-(J5-Pin_5): track 16.1 -> 12.7 mm
- net Net-(U1-BST): track 23.3 -> 20.2 mm
- net Net-(J5-Pin_6): track 17.0 -> 14.7 mm
- net RX: track 80.0 -> 81.7 mm, vias 5 -> 4
- net RST: track 47.8 -> 48.7 mm, vias 0 -> 1
- net Net-(Q1-C): track 17.3 -> 16.5 mm
- net Net-(U1-SW): track 3.17 -> 2.43 mm
- net Net-(BZ1--): track 10.4 -> 9.65 mm
- net Net-(Q2-E): track 16.4 -> 16.9 mm
- added copper zone on B.Cu, net GND

Commit message: Update symbol and footprint of WT8266
Parts:
- renumbered BATTERY to J2, KBD to J5, RFID to J6, TAMPER to SW1, TAMPER to TP1, GND to TP3, BUZZER to TP5
Routing:
- net GND: track 99.6 -> 76.4 mm, vias 2 -> 3
- net +12V: track 140.8 -> 143.3 mm
- net BUZZ: track 52.6 -> 54.9 mm
- net I2C_D: track 68.4 -> 69.5 mm
- added copper zone on F.Cu, net GND
