File: PIR/PIR.kicad_pcb (KiCad board)
At the start: 2 copper layers, 50 x 80 mm, 32 parts, among them J1 FLASH, J2 PIR, J3 BUS, J4 Conn_01x04_Socket, Q1 BC846, Q2 BC846, Q3 BC857, SW1 tamper switch, U1 AP63203WU, U2 WT8266-S1

Commit message: upgrades people, upgrades!
Routing:
- net +12V: track 173.7 -> 170.7 mm
Changed lines of the file:
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@@
   (segment (start 116.4381 75.4831) (end 115.955 75) (width 0.25) (layer "B.Cu") (net 2))
   (segment (start 110 79.755) (end 111.825 81.58) (width 0.25) (layer "B.Cu") (net 2))
-  (segment (start 133.74 126.74) (end 134.5 127.5) (width 0.25) (layer "F.Cu") (net 3))
   (segment (start 116.680698 56.5) (end 118.180698 58) (width 0.25) (layer "F.Cu") (net 3))
   (segment (start 137.6 93.1) (end 136.0175 93.1) (width 0.25) (layer "F.Cu") (net 3))
+  (segment (start 134 127) (end 142.5 127) (width 0.25) (layer "F.Cu") (net 3))
   (segment (start 138.5 94) (end 137.6 93.1) (width 0.25) (layer "F.Cu") (net 3))
-  (segment (start 133.74 124) (end 133.74 126.74) (width 0.25) (layer "F.Cu") (net 3))
+  (segment (start 143 125.1375) (end 143.9495 125.1375) (width 0.25) (layer "F.Cu") (net 3))
   (segment (start 145.5 125.1375) (end 143.95 125.1375) (width 0.25) (layer "F.Cu") (net 3))
   (segment (start 105.25 75.5) (end 102 72.25) (width 0.25) (layer "F.Cu") (net 3))
-  (segment (start 143 125.138) (end 143 125.1375) (width 0.25) (layer "F.Cu") (net 3))
-  (segment (start 143.5 127.5) (end 144 127) (width 0.25) (layer "F.Cu") (net 3))
   (segment (start 118.180698 58) (end 129.425 58) (width 0.25) (layer "F.Cu") (net 3))
+  (segment (start 133.74 124) (end 133.74 126.74) (width 0.25) (layer "F.Cu") (net 3))
   (segment (start 102 72.25) (end 102 64) (width 0.25) (layer "F.Cu") (net 3))
   (segment (start 145.5 125.825) (end 145.5 125.1375) (width 0.25) (layer "F.Cu") (net 3))
   (segment (start 145.675 126) (end 145.5 125.825) (width 0.25) (layer "F.Cu") (net 3))
   (segment (start 111.825 79.04) (end 108.285 75.5) (width 0.25) (layer "F.Cu") (net 3))
-  (segment (start 144 127) (end 144 125.188) (width 0.25) (layer "F.Cu") (net 3))
-  (segment (start 143 127.5) (end 143.5 127.5) (width 0.25) (layer "F.Cu") (net 3))
-  (segment (start 143 127.5) (end 143 125.138) (width 0.25) (layer "F.Cu") (net 3))
+  (segment (start 143 126.5) (end 143 125.1375) (width 0.25) (layer "F.Cu") (net 3))
   (segment (start 144 125.1875) (end 144 125.188) (width 0.25) (layer "F.Cu") (net 3))
   (segment (start 108.285 75.5) (end 105.25 75.5) (width 0.25) (layer "F.Cu") (net 3))
   (segment (start 129.425 58) (end 131.825 60.4) (width 0.25) (layer "F.Cu") (net 3))
   (segment (start 143.95 125.1375) (end 144 125.1875) (width 0.25) (layer "F.Cu") (net 3))
+  (segment (start 133.74 126.74) (end 134 127) (width 0.25) (layer "F.Cu") (net 3))
+  (segment (start 142.5 127) (end 143 126.5) (width 0.25) (layer "F.Cu") (net 3))
   (segment (start 135 105.5) (end 139.8 105.5) (width 0.25) (layer "F.Cu") (net 3))
   (segment (start 138.5 94.5) (end 138.5 94) (width 0.25) (layer "F.Cu") (net 3))
   (segment (start 148 126) (end 145.675 126) (width 0.25) (layer "F.Cu") (net 3))
+  (segment (start 143.9495 125.1375) (end 144 125.188) (width 0.25) (layer "F.Cu") (net 3))
   (segment (start 102 64) (end 109.5 56.5) (width 0.25) (layer "F.Cu") (net 3))
   (segment (start 109.5 56.5) (end 116.680698 56.5) (width 0.25) (layer "F.Cu") (net 3))
   (segment (start 133.74 106.76) (end 135 105.5) (width 0.25) (layer "F.Cu") (net 3))
-  (segment (start 134.5 127.5) (end 143 127.5) (width 0.25) (layer "F.Cu") (net 3))
   (segment (start 144 125.188) (end 144.132 125.32) (width 0.25) (layer "F.Cu") (net 3))
   (segment (start 133.74 124) (end 133.74 106.76) (width 0.25) (layer "F.Cu") (net 3))
@@
   (segment (start 143.925 119.575) (end 143 120.5) (width 1) (layer "F.Cu") (net 4))
   (segment (start 143 120.275) (end 143 122.8625) (width 0.5) (layer "F.Cu") (net 4))
-  (segment (start 142.05 122.8625) (end 142.05 121.1) (width 0.25) (layer "F.Cu") (net 5))
-  (segment (start 142.05 121.1) (end 141.45 120.5) (width 0.25) (layer "F.Cu") (net 5))
+  (segment (start 141.5 122.6) (end 141.5 120.55) (width 0.25) (layer "F.Cu") (net 5))
+  (segment (start 141.5 120.55) (end 141.45 120.5) (width 0.25) (layer "F.Cu") (net 5))
+  (segment (start 142.05 122.8625) (end 141.7625 122.8625) (width 0.25) (layer "F.Cu") (net 5))
+  (segment (start 141.7625 122.8625) (end 141.5 122.6) (width 0.25) (layer "F.Cu") (net 5))
   (segment (start 113.38 84.12) (end 111.825 84.12) (width 1) (layer "F.Cu") (net 6))
   (segment (start 126.413274 93.58) (end 125 93.58) (width 1) (layer "F.Cu") (net 6))
@@
   (segment (start 125 93.58) (end 123.58 93.58) (width 1) (layer "F.Cu") (net 6))
   (segment (start 115 83.5) (end 115 75.237792) (width 1) (layer "F.Cu") (net 6))
-  (segment (start 104.43 125.17) (end 104.43 118.67) (width 1) (layer "F.Cu") (net 6))
+  (segment (start 104.43 125.17) (end 104.43 118.67) (width 0.25) (layer "F.Cu") (net 6))
   (segment (start 106.5 64.5) (end 105.5 64.5) (width 1) (layer "F.Cu") (net 6))
   (segment (start 123.58 93.58) (end 119.38 89.38) (width 1) (layer "F.Cu") (net 6))
@@
   (segment (start 140 84.75) (end 140 82.5) (width 0.25) (layer "F.Cu") (net 13))
   (via (at 140 84.75) (size 0.8) (drill 0.4) (layers "F.Cu" "B.Cu") (net 13))
+  (segment (start 147.95 117.313604) (end 147.95 124.075305) (width 0.25) (layer "B.Cu") (net 13))
+  (segment (start 142.918442 129.106863) (end 125.106863 129.106863) (width 0.25) (layer "B.Cu") (net 13))
+  (segment (start 140 84.75) (end 140 109.363604) (width 0.25) (layer "B.Cu") (net 13))
+  (segment (start 125.106863 129.106863) (end 120 124) (width 0.25) (layer "B.Cu") (net 13))
   (segment (start 120 124) (end 118.74 124) (width 0.25) (layer "B.Cu") (net 13))
   (segment (start 140 109.363604) (end 147.95 117.313604) (width 0.25) (layer "B.Cu") (net 13))
-  (segment (start 143.200305 128.825) (end 124.825 128.825) (width 0.25) (layer "B.Cu") (net 13))
-  (segment (start 147.95 117.313604) (end 147.95 124.075305) (width 0.25) (layer "B.Cu") (net 13))
-  (segment (start 147.95 124.075305) (end 143.200305 128.825) (width 0.25) (layer "B.Cu") (net 13))
-  (segment (start 140 84.75) (end 140 109.363604) (width 0.25) (layer "B.Cu") (net 13))
-  (segment (start 124.825 128.825) (end 120 124) (width 0.25) (layer "B.Cu") (net 13))
+  (segment (start 147.95 124.075305) (end 142.918442 129.106863) (width 0.25) (layer "B.Cu") (net 13))
   (segment (start 126 79) (end 126 76) (width 0.25) (layer "F.Cu") (net 14))
   (segment (start 137 66) (end 136 65) (width 0.25) (layer "F.Cu") (net 14))
