File: Universal module/PIR systém Q.kicad_pcb (KiCad board)
At the start: 2 copper layers, 50 x 80 mm, 32 parts, among them J1 FLASH, J2 PIR, J3 BUS, J4 Conn_01x04_Socket, Q1 BC846, Q2 BC846, Q3 BC857, SW1 tamper switch, U1 AP63203WU, U2 WT8266-S1

Commit message: begun the drawing of the PCB, fixed libraries
Parts:
- removed J2: PIR, Connector_PinSocket_2.54mm:PinSocket_1x03_P2.54mm_Vertical
- removed J3: BUS, TerminalBlock:TerminalBlock_Altech_AK300-4_P5.00mm
- removed R7: 10k, Resistor_SMD:R_0603_1608Metric
- added C6: 100nF, Capacitor_SMD:C_0603_1608Metric, F.Cu at (74.9, 69.7)
- added C7: 100nF, Capacitor_SMD:C_0603_1608Metric, F.Cu at (74.9, 72.2)
- added D2: D, Diode_SMD:D_0603_1608Metric, F.Cu at (90.6, 47.9)
- added D4: D, Diode_SMD:D_0603_1608Metric, F.Cu at (90.6, 50.5)
- added J5: USB_B_Mini, Connector_USB:USB_Mini-B_Tensility_54-00023_Vertical, F.Cu at (106.5, 58.6)
- added Q4: BC817, Package_TO_SOT_SMD:SOT-23, F.Cu at (51.4, 74.7)
- added Q5: BC817, Package_TO_SOT_SMD:SOT-23, F.Cu at (51.4, 79.3)
- added R10: 10k, Resistor_SMD:R_0603_1608Metric, F.Cu at (82.9, 64.7)
- added R11: 10k, Resistor_SMD:R_0603_1608Metric, F.Cu at (82.9, 67.2)
- added R12: 10k, Resistor_SMD:R_0603_1608Metric, F.Cu at (82.9, 69.7)
- added R8: 10k, Resistor_SMD:R_0603_1608Metric, F.Cu at (82.9, 59.7)
- added R9: 10k, Resistor_SMD:R_0603_1608Metric, F.Cu at (82.9, 62.2)
- added U3: CH340C, Package_SO:SOIC-16_3.9x9.9mm_P1.27mm, F.Cu at (108.0, 69.7)
- added U4: P82B96, P82B96D:SOIC127P599X175-8N, F.Cu at (125.0, 132.4)
- BZ1: footprint LPT2270AS buzzer:LPT2270AS -> piezo:LPT2270AS
- J1: value FLASH -> Screw_Terminal_01x06; footprint Connector_PinSocket_2.54mm:PinSocket_1x06_P2.54mm_Horizontal -> TerminalBlock_Phoenix:TerminalBlock_Phoenix_MKDS-1,5-6_1x06_P5.00mm_Horizontal
- moved R2 91.5 mm to (78.9, 62.2), turned to 0 degrees
- moved C2 91.1 mm to (74.9, 59.7), turned to 0 degrees
- moved Q1 88.2 mm to (51.4, 60.8)
- moved Q2 88.1 mm to (51.4, 65.5)
- moved Q3 88.1 mm to (51.4, 70.1)
- moved J1 86.6 mm to (113.2, 145.0), turned to 0 degrees
- moved TP3 84.9 mm to (86.7, 67.3), turned to 0 degrees
- moved R1 64.7 mm to (78.9, 59.7), turned to 0 degrees
- moved D1 62.7 mm to (65.3, 83.8)
- moved TP5 60.1 mm to (90.2, 60.2)
- moved TP6 59.8 mm to (90.2, 63.8), turned to 0 degrees
- moved R3 58.6 mm to (78.9, 64.7), turned to 0 degrees
- moved TP4 57.6 mm to (86.7, 70.9)
- moved TP2 53.5 mm to (86.7, 63.8)
- moved R4 52.3 mm to (78.9, 67.2), turned to 0 degrees
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Connections:
- C5 pad 1: "reset" -> ESP_EN
- J1 pad 1: +12V -> Net-(D4-A)
- J1 pad 2: TX -> GND
- J1 pad 3: RX -> SDA
- J1 pad 4: GPIO0 -> SCL
- J1 pad 5: GND -> +3.3V
- J1 pad 6: "reset" -> PIR Signal
- R5 pad 1: "reset" -> ESP_EN
- TP1 pad 1: PIR signal -> PIR Signal
- TP5 pad 1: "reset" -> ESP_EN
- U2 pad 14: "reset" -> ESP_EN
Routing:
- net GND: track 278.0 -> 0.00 mm, vias 3 -> 0
- net +3.3V: track 222.0 -> 0.00 mm, vias 16 -> 0
- net +12V: track 169.9 -> 0.00 mm, vias 1 -> 0
- net tamper: track 107.4 -> 0.00 mm, vias 2 -> 0
- net "reset": track 84.4 -> 0.00 mm, vias 3 -> 0
- net I2C data: track 77.7 -> 0.00 mm, vias 4 -> 0
- net clock: track 63.9 -> 0.00 mm, vias 1 -> 0
- net PIR signal: track 59.5 -> 0.00 mm, vias 2 -> 0
- net Net-(Q1-C): track 53.3 -> 0.00 mm, vias 5 -> 0
- net Net-(D1-A): track 51.8 -> 0.00 mm, vias 3 -> 0
- net battery voltage: track 51.5 -> 0.00 mm, vias 5 -> 0
- net GPIO0: track 27.3 -> 0.00 mm, vias 2 -> 0
- net TX: track 23.1 -> 0.00 mm, vias 2 -> 0
- net Net-(BZ1--): track 23.0 -> 0.00 mm
- net Net-(Q2-E): track 21.5 -> 0.00 mm, vias 2 -> 0
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Other:
- board size 50 x 80 mm -> 50 x 100 mm
- board text removed: "+12V"
- board text removed: "+3.3V"
- board text removed: "12V"
- board text removed: ":3"
- board text removed: "BATT. V"
- board text removed: "BUZZER"
- board text removed: "CLOCK"
- board text removed: "GND"
- board text removed: "GPIO 0"
- board text removed: "HW. Rev. 1 Q PIR 24.8.2023"
- board text removed: "I2C DATA"
- board text removed: "PIR"
- board text removed: "PIR LED"
- board text removed: "RESET"
- board text removed: "RX"
- board text removed: "TAMPER T."
- board text removed: "TX"
- board text removed: "Tamper"
- board text removed: "V ms."

Commit message: basic PCB design
Parts:
- BATT V.: renamed from TP6
- Buzzer : renamed from TP4
- I2C convertor: renamed from U4
- USB UART: renamed from J5
- moved PIR 103.4 mm to (146.7, 144.5)
- moved Q1 93.8 mm to (133.5, 106.0)
- moved Q4 92.8 mm to (142.2, 93.6)
- moved Q5 92.8 mm to (142.2, 98.2)
- moved C2 91.6 mm to (146.6, 116.8), turned to 90 degrees
- moved Q2 87.9 mm to (129.4, 106.0)
- moved Q3 82.2 mm to (125.3, 106.0)
- moved GND 72.7 mm to (117.1, 134.8)
- moved R2 72.2 mm to (132.8, 110.3)
- moved Tamper 71.7 mm to (145.3, 74.3), turned to 180 degrees
- moved C4 71.5 mm to (142.8, 87.0)
- moved C5 71.4 mm to (142.8, 89.2)
- moved C3 69.2 mm to (138.6, 89.2)
- moved C6 66.1 mm to (138.6, 87.1)
- moved R9 65.0 mm to (137.7, 97.2), turned to -90 degrees
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- renumbered TP3 to 12V, U3 to CH340, U2 to ESP8266, TP5 to ESP_EN, TP7 to GND, D1 to LED, TP1 to PIR, BZ1 to Piezo, U1 to Regulator, SW1 to Tamper
Connections:
- ESP8266 pad 19: (no net) -> GND
- ESP8266 pad 2: PIR signal -> PIR Signal
Routing:
- net GND: track 0.00 -> 293.9 mm, vias 0 -> 8
- net +3.3V: track 0.00 -> 188.7 mm, vias 0 -> 5
- net +12V: track 0.00 -> 121.7 mm, vias 0 -> 4
- net PIR Signal: track 0.00 -> 117.7 mm, vias 0 -> 5
- net clock: track 0.00 -> 110.8 mm
- net I2C data: track 0.00 -> 100.2 mm, vias 0 -> 3
- net Net-(D4-A): track 0.00 -> 85.1 mm
- net GPIO0: track 0.00 -> 53.4 mm, vias 0 -> 2
- net Net-(Q1-B): track 0.00 -> 50.4 mm, vias 0 -> 4
- net Net-(Q5-E): track 0.00 -> 44.8 mm, vias 0 -> 2
- net Net-(Q4-E): track 0.00 -> 42.7 mm
- net ESP_EN: track 0.00 -> 42.3 mm, vias 0 -> 2
- net battery voltage: track 0.00 -> 35.0 mm, vias 0 -> 4
- net Net-(Q1-C): track 0.00 -> 31.2 mm, vias 0 -> 2
- net TX: track 0.00 -> 29.1 mm
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Other:
- board text added: "+12V"
- board text added: "+3,3V"
- board text added: "Despite his criminal mind, this man is behaving well. His reward is the canoe. This time, he can sit in the canoe for up to an hour."
- board text added: "GND"
- board text added: "PIR"
- board text added: "SCL"
- board text added: "SDA"

Commit message: finish PCB design, bonus gerber files
Parts:
- removed PIR: 3,3V, TestPoint:TestPoint_Pad_1.5x1.5mm
- added KB: Conn_01x04_Socket, Connector_PinSocket_2.54mm:PinSocket_1x04_P2.54mm_Vertical, F.Cu at (106.8, 85.1)
- BATT: renamed from J4; footprint Connector_PinSocket_2.54mm:PinSocket_1x04_P2.54mm_Horizontal -> Connector_PinSocket_2.54mm:PinSocket_1x04_P2.54mm_Vertical
- BATT: renamed from BATT V.
- Siren: renamed from Buzzer 
- Siren: renamed from Piezo; value Buzzer -> Siren
- U4: renamed from I2C convertor
- USB: renamed from USB UART
- moved 12V 31.7 mm to (129.4, 117.2)
- moved GND 12.6 mm to (106.2, 141.2)
- moved Q1 3.84 mm to (137.3, 105.6)
- moved Q2 3.84 mm to (133.2, 105.6)
- moved Q3 3.84 mm to (129.1, 105.6)
- moved R2 3.84 mm to (136.6, 109.8)
- moved R3 3.84 mm to (127.4, 101.7)
- moved BATT 2.00 mm to (117.7, 83.2)
- moved J1 0.76 mm to (112.5, 144.9)
- moved BATT 0.22 mm to (113.3, 85.1)
- renumbered Tamper to TAMPER, TP2 to TAMPER, Regulator to U1
Connections:
- ESP8266 pad 19: GND -> (no net)
Routing:
- net GPIO0: track 53.4 -> 96.0 mm, vias 2 -> 5
- net RX: track 22.0 -> 56.4 mm, vias 0 -> 3
- net TX: track 29.1 -> 53.1 mm, vias 0 -> 2
- net Net-(Q1-C): track 31.2 -> 15.1 mm, vias 2 -> 0
- net PIR Signal: track 117.7 -> 132.9 mm, vias 5 -> 4
- net GND: track 293.9 -> 284.8 mm, vias 8 -> 10
- net Net-(U2-GPIO5): track 24.2 -> 17.7 mm, vias 0 -> 2
- net +12V: track 121.7 -> 125.8 mm
- net Net-(BZ1--): track 25.5 -> 29.6 mm, vias 2 -> 4
- net Net-(J5-D-): track 23.8 -> 27.1 mm
- net Net-(Q2-E): track 17.0 -> 14.2 mm, vias 3 -> 2
- net Net-(Q1-B): track 50.4 -> 47.9 mm
- net battery voltage: track 35.0 -> 37.1 mm
- net +3.3V: track 188.7 -> 186.8 mm
- net Net-(Q4-E): track 42.7 -> 44.4 mm
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- added copper zone on B.Cu, net GND
- added copper zone on F.Cu, net GND
Other:
- outline, holes or cut-outs redrawn
- board text added: ":3"
- board text added: "HW. Rev. 2 Q Universal module 3.12.2024"

Commit message: fix small issues
Parts:
- moved Siren 1.23 mm to (113.4, 111.7)
Connections:
- ESP8266 pad 19: (no net) -> GND
Routing:
- net GND: track 284.8 -> 274.1 mm, vias 10 -> 12
- net +3.3V: track 186.8 -> 185.6 mm
